Commit message: update urdf to include visual model

File: bluerov_robot/urdf/bluerov.urdf (robot description, URDF)
Before this commit: robot bluerov, 3 links, 2 joints
Links:
- removed link fcu
- removed link thruster0
- link base_link: geometry visual mesh filename=package://bluerov_robot/robot/bluerov2.dae
Joints:
- removed joint base_link_to_fcu
- removed joint base_link_to_thruster0
